File: anavi-miracle-uhat.kicad_pcb (KiCad board)
At the start: 2 copper layers, 65 x 30 mm, 25 parts, among them U1 CAT24C32WI-GT3, U2 74LVC1G17W5-7

Commit message: anavi-miracle-uhat: Add assembly notes
Add assembly notes to the front fabrication layer.

Signed-off-by: Leon Anavi <leon@anavi.org>
Other:
- board text removed: "100nF"
Changed lines of the file:
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@@
       (effects (font (size 0.6 0.6) (thickness 0.1)))
     )
-    (fp_text value "4.7K" (at 0 1.9) (layer "F.Fab")
+    (fp_text value "4.7K" (at -0.016 -2.292) (layer "F.Fab")
       (effects (font (size 1 1) (thickness 0.15)))
     )
@@
       (effects (font (size 0.6 0.6) (thickness 0.1)))
     )
-    (fp_text value "4.7K" (at 0 1.9) (layer "F.Fab")
+    (fp_text value "4.7K" (at 0.026 -2.292) (layer "F.Fab")
       (effects (font (size 1 1) (thickness 0.15)))
     )
@@
     (effects (font (size 0.8 0.8) (thickness 0.2)))
   )
-  (gr_text "4,7K" (at 203.9 83.9) (layer "F.Fab")
+  (gr_text "4,7K" (at 206.36 85.5) (layer "F.Fab")
     (effects (font (size 1 1) (thickness 0.25)))
   )
-  (gr_text "1K" (at 210 88.9 90) (layer "F.Fab")
+  (gr_text "1K" (at 211.6 88.95 90) (layer "F.Fab")
     (effects (font (size 1 1) (thickness 0.25)))
   )
-  (gr_text "100nF" (at 210 83.9 90) (layer "F.Fab")
-    (effects (font (size 1 0.8) (thickness 0.2)))
-  )
-  (gr_text "4,7K" (at 203.9 87.9) (layer "F.Fab")
+  (gr_text "4,7K" (at 206.44 90.74) (layer "F.Fab")
     (effects (font (size 1 1) (thickness 0.25)))
   )
